Commit message: Añadido LIDAR a dron firefly
Se añade LIDAR Ouster OS-1 al dron firefly de rotorS. He hecho pruebas para moverlo en velocidad pero no lo he logrado, de momento sólo lo sé mover en posición.

File: catkin_ws/src/rotors_simulator/rotors_description/urdf/firefly_base.xacro (robot description, xacro)
@@ -41,3 +41,7 @@
       wait_to_record_bag="$(arg wait_to_record_bag)" />
   </xacro:if>
+	<xacro:include filename="$(find rotors_description)/urdf/OS1-64.urdf.xacro"/>
+  <OS1-64 parent="${namespace}/base_link" name="${namespace}/os1_sensor" hz="10" samples="220">
+    <origin xyz="0 0 -0.0365" rpy="0 0 0" />
+  </OS1-64>
 </robot>

Commit message: Añadidas simulaciones y cambios varios.
Se hacen los ficheros .launch de los experimentos, además se añaden nuevos ficheros .cpp para controlar los drones. Los ficheros .launch se han hecho de forma que se pueda seleccionar la velocidad de los drones al lanzarlo. Por ejemplo, roslaunch mis_programas experimento_2.launch max_vel_1:=1.0 max_vel_2:=-1.0
max_vel_1 hace referencia al dron con el LIDAR y max_vel_2 al otro.
Se añade el directorio urdf. Ahora el LIDAR se añade sin modificar los paquetes originales de rotorS ni los de ouster, si no que, se llaman desde los distintos ficheros.

File: catkin_ws/src/rotors_simulator/rotors_description/urdf/firefly_base.xacro (robot description, xacro)
@@ -41,7 +41,3 @@
       wait_to_record_bag="$(arg wait_to_record_bag)" />
   </xacro:if>
-   <xacro:include filename="$(find rotors_description)/urdf/OS1-64.urdf.xacro"/>
-  <OS1-64 parent="${namespace}/base_link" name="${namespace}/os1_sensor" hz="10" samples="220">
-    <origin xyz="0 0 -0.0365" rpy="0 0 0" />
-  </OS1-64>
 </robot>
